Commit message: modified extended body lift

File: hexapod_description/urdf/razbot_model.xacro (robot description, xacro)
@@ -18,5 +18,5 @@
         <parent link="base_link" />
         <child link="body_link" />
-        <origin xyz="0.0 0.0 0.0" rpy="0.0 0.0 0.0" />
+        <origin xyz="0.0 0.0 0.065" rpy="0.0 0.0 0.0" />
     </joint>
 	<link name="body_link">
@@ -55,5 +55,5 @@
 		<parent link="base_link" />
 		<child link="imu_link" />
-		<origin xyz="0.0 0.0 0.0" rpy="0.0 0.0 0.0" />
+		<origin xyz="0.0 0.0 0.092" rpy="0.0 0.0 -${pi/2}" />
 	</joint>
 	<link name="imu_link">
@@ -190,5 +190,5 @@
 		<!-- tibia -->
 		<joint name="tibia_joint_${side}${position}" type="revolute">
-			<origin xyz="0.0 -${femur_length} 0.0" rpy="${pi} 0.0 0.0" />
+			<origin xyz="-0.004 -${femur_length} 0.0" rpy="${pi} 0.0 0.0" />
 			<parent link="femur_${side}${position}" />
 			<child link="tibia_${side}${position}" />
@@ -236,4 +236,29 @@
         <gazebo reference="tibia_${side}${position}">
             <material>Gazebo/DarkGrey</material>
+        </gazebo>
+                <!-- foot -->
+        <joint name="foot_joint_${side}${position}" type="fixed">
+            <origin xyz="${tibia_length} 0.025 0.0" rpy="0.0 0.0 0.0" />
+            <parent link="tibia_${side}${position}" />
+            <child link="foot_${side}${position}" />
+        </joint>
+        <link name="foot_${side}${position}">
+            <inertial>
+                <origin xyz="0.0 0.0 0.0" rpy="0.0 0.0 0.0" />
+                <mass value="0.00001"/>
+                <inertia
+                    ixx="1.0" ixy="0.0"  ixz="0.0"
+                    iyy="1.0" iyz="0.0"
+                    izz="1.0" />
+            </inertial>
+        </link>
+        <gazebo>
+            <plugin name="f3d_controller" filename="libgazebo_ros_f3d.so">
+                <alwaysOn>true</alwaysOn>
+                <updateRate>50</updateRate>
+                <bodyName>foot_${side}${position}</bodyName>
+                <topicName>${side}${position}_ground_feedback</topicName>
+                <frameName>foot_${side}${position}</frameName>
+            </plugin>
         </gazebo>
 	</xacro:macro>

Commit message: second commit

File: hexapod_description/urdf/razbot_model.xacro (robot description, xacro)
@@ -18,5 +18,5 @@
         <parent link="base_link" />
         <child link="body_link" />
-        <origin xyz="0.0 0.0 0.065" rpy="0.0 0.0 0.0" />
+        <origin xyz="0.0 0.0 0.024" rpy="0.0 0.0 0.0" />
     </joint>
 	<link name="body_link">
@@ -51,9 +51,40 @@
         <material>Gazebo/DarkGrey</material>
     </gazebo>
+		<!-- Camera properties -->
+    <joint name="camera_rgb_joint" type="fixed">
+        <parent link="body_link"/>
+        <child link="camera_rgb_optical_frame"/>
+        <origin xyz="0.05 -0.015 0.099" rpy="${pi/2} ${pi} ${pi/2}"/>
+    </joint>
+    <link name="camera_rgb_optical_frame">
+        <inertial>
+            <origin xyz="0.0 0.0 0.0" rpy="0.0 0.0 0.0" />
+            <mass value="0.00001"/>
+            <inertia
+                ixx="1.0" ixy="0.0"  ixz="0.0"
+                iyy="1.0" iyz="0.0"
+                izz="1.0" />
+        </inertial>
+    </link>
+    <joint name="camera_depth_joint" type="fixed">
+        <parent link="body_link"/>
+        <child link="camera_depth_optical_frame"/>
+        <origin xyz="0.05 0.015 0.099" rpy="${pi/2} ${pi} ${pi/2}"/>
+    </joint>
+    <link name="camera_depth_optical_frame">
+        <inertial>
+            <origin xyz="0.0 0.0 0.0" rpy="0.0 0.0 0.0" />
+            <mass value="0.00001"/>
+            <inertia
+                ixx="1.0" ixy="0.0"  ixz="0.0"
+                iyy="1.0" iyz="0.0"
+                izz="1.0" />
+        </inertial>
+		</link>
 	<!-- IMU properties -->
 	<joint name="imu_joint" type="fixed">
-		<parent link="base_link" />
+		<parent link="body_link" />
 		<child link="imu_link" />
-		<origin xyz="0.0 0.0 0.092" rpy="0.0 0.0 -${pi/2}" />
+		<origin xyz="0.0 0.0 0.021" rpy="0.0 0.0 -${pi/2}" />
 	</joint>
 	<link name="imu_link">
